File: Hardware/PCB/core stage.kicad_sch (KiCad schematic)
At the start: 24 parts, among them IC8 ATXMEGA32A4U

Commit message: Implemented the new hardware features
Co-Authored-By: David Palma <78764277+davidpalma666@users.noreply.github.com>
Parts:
- C13: footprint FastStepper PCBLib:C0402K -> Capacitor_SMD:C_0402_1005Metric; OEPS OEPS010011 -> (none); OEPSPN (none) -> OEPS010011
- C15: footprint FastStepper PCBLib:C0603K -> Capacitor_SMD:C_0603_1608Metric; MPN DNI -> n.a.; OEPS DNI -> (none); OEPSPN (none) -> n.a.; now not fitted
- C16, C25, C26, C27, C28, C29: footprint FastStepper PCBLib:C0402K -> Capacitor_SMD:C_0402_1005Metric; MPN C1005X7R1H104K050BB -> CGA2B3X7R1H104K050BB; OEPS OEPS010004 -> (none); OEPSPN (none) -> OEPS010016
- IC8: footprint FastStepper PCBLib:TQFP44 -> Package_QFP:TQFP-44_10x10mm_P0.8mm; MPN ATXMEGA32A4U-AUR -> ATXMEGA32A4U-A; OEPS OEPS080012 -> (none); OEPSPN (none) -> OEPS080012
- L2, L3: footprint FastStepper PCBLib:R0805 -> Resistor_SMD:R_0805_2012Metric; OEPS OEPS040003 -> (none); OEPSPN (none) -> OEPS040003
- R1: footprint FastStepper PCBLib:R0402 -> Resistor_SMD:R_0402_1005Metric; OEPS OEPS020037 -> (none); OEPSPN (none) -> OEPS020037
- R34: footprint FastStepper PCBLib:R0402 -> Resistor_SMD:R_0402_1005Metric; MPN CRCW040210K0FKED -> ERJ-2RKF1002X; OEPS OEPS020030 -> (none); OEPSPN (none) -> OEPS020013
- R4, R7, R9: footprint FastStepper PCBLib:R0402 -> Resistor_SMD:R_0402_1005Metric; MPN DNI -> n.a.; OEPS DNI -> (none); OEPSPN (none) -> n.a.; now not fitted
- STATE0: footprint FastStepper PCBLib:CHIP-LED0603 -> LED_SMD:LED_0603_1608Metric; OEPS OEPS030005 -> (none); OEPSPN (none) -> OEPS030005
- SV2: footprint FastStepper PCBLib:2X03 -> Connector_PinHeader_2.54mm:PinHeader_2x03_P2.54mm_Vertical; MPN 609-3210-ND -> PR20203VBDN; OEPS OEPS070015 -> (none); OEPSPN (none) -> OEPS070124
- TP4, TP5, TP6, TP8, TP9: footprint FastStepper PCBLib:TP11R -> TestPoint:TestPoint_THTPad_D1.0mm_Drill0.5mm; now left out of the parts list
- X6: renamed from OSC1; footprint FastStepper PCBLib:OSCILLATOR_3.2X2.5 -> Oscillator:Oscillator_SMD_Abracon_ASE-4Pin_3.2x2.5mm; OEPS OEPS080018 -> (none); OEPSPN (none) -> OEPS080018
Connections:
- net +3.3V_u: now also X6.4 (VDD); no longer X6.P$4 (VDD)
- net GND: now also X6.2 (GND); no longer X6.P$2 (GND)
- net at IC8.37 (PR1/XTAL1): now also X6.3 (OUTPUT); no longer X6.P$3 (OUTPUT)
- net U_CLOCK_IN renamed CLK_2u
Other:
- moved on the sheet: L2
